File: circuit/Mozard Nano.brd (EAGLE design)
At the start: 69.8 x 67.3 mm, 22 parts, among them J2 SPKR, J3 OUT, U2 LM386

Commit message: Fixes and added other potentiometer
Parts:
- added JP1: RX, TOF:1X01_SIDE_NAME
- added JP2: TX, TOF:1X01_SIDE_NAME
- added JP3: GND, TOF:1X01_SIDE_NAME
- added POT6: 10K, SparkFun-Electromechanical:ALPS_POT_KIT
- R4, R6, R7: device adafruit:0204/5 -> adafruit:0204/7
- moved C2 10.2 mm to (40.6, 29.2)
- moved R7 10.2 mm to (33.0, 39.4)
- moved C4 9.16 mm to (33.0, 29.2)
- moved C1 8.52 mm to (33.0, 33.0)
- moved R6 7.62 mm to (33.0, 41.9)
- moved U$2 7.18 mm to (54.4, 30.0)
- moved C_AMP 6.35 mm to (45.7, 47.0)
- moved U2 3.81 mm to (34.3, 48.3)
- moved R4 2.54 mm to (33.0, 36.8)
- renumbered POT to POT7
Connections:
- net POT renamed POT7
- removed net A6: KB1.C, U$1.A6
- removed net N$5: C2.2, OUT_VOLUME.P$1
- new net A1: KB1.C, U$1.A1
- new net N$2: C2.2, OUT_VOLUME.P$3
- new net POT6: POT6.P$2, U$1.A6
- new net RX: JP1.1, U$1.RX1
- new net TX: JP2.1, U$1.TX0
- net GND: now also JP3.1, OUT_VOLUME.P$1, POT6.P$1, POT7.P$1; no longer OUT_VOLUME.P$3, POT7.P$3
- net VCC: now also POT6.P$3, POT7.P$3; no longer POT7.P$1
Routing:
- net GND: track 0.00 -> 111.3 mm
- net A1: track 0.00 -> 38.2 mm
- net POT6: track 0.00 -> 31.9 mm
- net N$5: track 30.5 -> 0.00 mm
- net N$2: track 0.00 -> 28.7 mm
- net A6: track 28.3 -> 0.00 mm
- net TX: track 0.00 -> 25.5 mm
- net RX: track 0.00 -> 25.5 mm
- net N$8: track 49.0 -> 30.2 mm
- net N$1: track 36.7 -> 18.4 mm
- net D9(AUDIO3.9K): track 31.3 -> 20.6 mm, vias 1 -> 0
- net VCC: track 60.0 -> 70.4 mm
- net D10(AUDIO499K): track 28.8 -> 20.6 mm
- net N$4: track 15.0 -> 20.4 mm
- net UNFILTERED_OUT: track 20.2 -> 15.1 mm
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Other:
- board text added: "Mozard 2018-05-15 by tofstuff.com"
- board text removed: "1"
- board text removed: "Mozard Nano by tofstuff.com"
