File: circuit/Mozard Nano.sch (EAGLE design)
At the start: 22 parts, among them J2 SPKR, J3 OUT, U2 LM386

Commit message: Fixes and added other potentiometer
Parts:
- removed POT: 10K, SparkFun-Electromechanical:POTALPS-KIT
- added JP1: RX, TOF:HEADER-1X1
- added JP2: TX, TOF:HEADER-1X1
- added JP3: GND, TOF:HEADER-1X1
- added POT6, POT7: 10K, SparkFun-Electromechanical:POTALPS-KIT
- R4, R6, R7: device adafruit:R-US_0204/5 -> adafruit:R-US_0204/7
Connections:
- removed net A6: KB1.C, U$1.A6
- removed net N$5: C2.2, OUT_VOLUME.E
- removed net POT: POT.S, U$1.A7
- new net A1: KB1.C, U$1.A1
- new net N$2: C2.2, OUT_VOLUME.A
- new net POT6: POT6.S, U$1.A6
- new net POT7: POT7.S, U$1.A7
- new net RX: JP1.1, U$1.RX1
- new net TX: JP2.1, U$1.TX0
- net GND: now also JP3.1, OUT_VOLUME.E, POT6.E, POT7.E; no longer OUT_VOLUME.A, POT.A
- net VCC: now also POT6.A, POT7.A; no longer POT.E
Other:
- moved on the sheet: OUT_VOLUME
