File: extras/circuit/Mozard 2020-10-18.brd (EAGLE design)
At the start: 94 x 71.1 mm, 42 parts, among them J4 Headphone/Line Out, U2 LM386

Commit message: New version
Parts:
- removed R5: 270, adafruit:0204/5
- added C_AMP: 100uF, Mitch-parts:CPOL-RADIAL-10UF-25V
- added JP1: TX, TOF:1X01_SIDE_NAME
- moved R1 9.26 mm to (41.9, 45.1), turned to 180 degrees
- moved C2 8.18 mm to (47.6, 33.7)
- moved C1 3.33 mm to (40.0, 33.7)
- moved R4 3.17 mm to (41.9, 37.5)
- moved R6 3.17 mm to (41.9, 42.5)
- moved R7 3.17 mm to (41.9, 40.0)
- moved C4 2.69 mm to (40.0, 30.2)
- moved SP1 2.42 mm to (63.8, 44.8)
- moved JP2 0.95 mm to (10.5, 68.6)
- moved JP5 0.95 mm to (13.0, 68.6)
- moved U2 0.63 mm to (42.5, 52.1)
- renumbered A1 to OCTAVE, A6 to T, A7 to PARAM
Connections:
- removed net LM386_OUTPUT: SP1.+, U2.5
- new net N$1: C_AMP.+, U2.5
- new net N$5: C_AMP.-, SP1.+
- net RX: no longer R5.2
- net TX: now also JP1.1
- net VCC: no longer R5.1
Routing:
- net TX: track 0.00 -> 48.9 mm, vias 0 -> 2
- net GND: track 237.3 -> 208.4 mm
- net N$5: track 0.00 -> 21.9 mm
- net N$1: track 0.00 -> 20.3 mm
- net LM386_OUTPUT: track 13.4 -> 0.00 mm
- net N$4: track 16.2 -> 10.0 mm
- net VCC: track 190.0 -> 186.3 mm
- net D9(AUDIO3.9K): track 18.2 -> 21.8 mm
- net D10(AUDIO499K): track 18.2 -> 21.6 mm
- net N$6: track 22.7 -> 25.2 mm
- net N$2: track 48.1 -> 46.5 mm
- net RX: track 73.9 -> 72.4 mm
Other:
- board text added: "ARP"
- board text added: "AUDIO OUT"
- board text added: "JLCJLCJLCJLC"
- board text added: "LAY 100uF CAP SIDEWAYS HERE"
- board text added: "MIDI IN"
- board text added: "MODE"
- board text added: "MOZARD 2020-10-18 TOFSTUFF.COM"
- board text added: "SPKR-"
- board text added: "|-|--|----|"
- board text removed: "M4"
- board text removed: "M5"
- board text removed: "MOZARD 2019-09-19 TOFSTUFF.COM"
