File: extras/circuit/Mozard 2020-10-18.sch (EAGLE design)
At the start: 42 parts, among them J4 Headphone/Line Out, U2 LM386

Commit message: New version
Parts:
- removed A1: A1, TOF:POT
- removed A6: A6, TOF:POT
- removed A7: A7, TOF:POT
- removed R5: 270, adafruit:R-US_0204/5
- added C_AMP: 100uF, Mitch-parts:CPOL-RADIAL-10UF-25V
- added JP1: TX, TOF:HEADER-1X1
- added OCTAVE: A1, TOF:POT
- added PARAM: A7, TOF:POT
- added T: A6, TOF:POT
Connections:
- removed net LM386_OUTPUT: SP1.+, U2.OUT
- new net N$1: C_AMP.+, U2.OUT
- new net N$5: C_AMP.-, SP1.+
- net A1: now also OCTAVE.S; no longer A1.S
- net A6: now also T.S; no longer A6.S
- net A7: now also PARAM.S; no longer A7.S
- net GND: now also OCTAVE.E, PARAM.E, T.E; no longer A1.E, A6.E, A7.E
- net RX: no longer R5.2
- net TX: now also JP1.1
- net VCC: now also OCTAVE.A, PARAM.A, T.A; no longer A1.A, A6.A, A7.A, R5.1
Other:
- note added: "Disabled when there is a connector"
- note removed: "CHANGES 2018-08-01 - updated labels and exposed rx"
- note removed: "How to disable MIDI IN when a jack is not connected? Because it disables the Arduino reprogramming :("
- note removed: "Silent when connector"
- moved on the sheet: 1N4148, C1, C2, C4, H1, H2, H3, H4, H5, H6, J4, JP2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
