File: extras/circuit/Mozard.brd (EAGLE design)
At the start: 94 x 71.1 mm, 43 parts, among them J4 Headphone/Line Out, U2 LM386

Commit message: Documentation
Parts:
- R1: value 100k -> 3.9k
Changed lines of the file:
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@@
 <element name="U$13" library="TOF" package="PCB-TOUCHPAD-1-PIN" value="PCB-TOUCHPAD-1-PIN" x="77.47" y="6.35" smashed="yes" rot="R270"/>
 <element name="U$14" library="TOF" package="PCB-TOUCHPAD-1-PIN" value="PCB-TOUCHPAD-1-PIN" x="88.9" y="15.24" smashed="yes" rot="R270"/>
-<element name="R1" library="adafruit" package="0204/7" value="100k" x="41.91" y="45.085" smashed="yes" rot="R180">
+<element name="R1" library="adafruit" package="0204/7" value="3.9k" x="41.91" y="45.085" smashed="yes" rot="R180">
 <attribute name="NAME" x="44.45" y="43.7896" size="0.9906" layer="25" ratio="12" rot="R180"/>
 <attribute name="VALUE" x="39.6494" y="44.2849" size="1.27" layer="27" ratio="12"/>
