File: extras/circuit/Mozard.sch (EAGLE design)
At the start: 43 parts, among them J4 Headphone/Line Out, U2 LM386

Commit message: Documentation
Parts:
- R1: value 100k -> 3.9k
Other:
- note added: "CHANGES: -2024/09/03: Changed R1 from 100k to 3.9k to reduce noise when speaker is not used"
Changed lines of the file:
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@@
 <part name="U$13" library="TOF" deviceset="PCB-TOUCHPAD-1-PIN" device=""/>
 <part name="U$14" library="TOF" deviceset="PCB-TOUCHPAD-1-PIN" device=""/>
-<part name="R1" library="adafruit" deviceset="R-US_" device="0204/7" value="100k"/>
+<part name="R1" library="adafruit" deviceset="R-US_" device="0204/7" value="3.9k"/>
 <part name="SUPPLY3" library="SparkFun-Aesthetics" deviceset="VCC" device=""/>
 <part name="SUPPLY7" library="SparkFun-Aesthetics" deviceset="VCC" device=""/>
@@
 <text x="177.8" y="139.7" size="1.778" layer="97">LOP Filter and Buffer</text>
 <text x="152.4" y="189.23" size="1.778" layer="97">MOZZI PWM</text>
+<text x="7.62" y="208.28" size="1.778" layer="97" align="top-left">CHANGES:
+-2024/09/03: Changed R1 from 100k to 3.9k to reduce noise when speaker is not used</text>
 </plain>
 <instances>
